Commit message: Unify robot description and organize control namespaces

File: src/wanren_arm/urdf/wanren_arm.urdf (robot description, URDF)
Before this commit: robot wanren_arm, 15 links, 14 joints
Links:
- added link arm_left_link_1, mass 0.120; collision cylinder length=0.180 radius=0.025; visual cylinder length=0.180 radius=0.025
- added link arm_left_link_2, mass 0.120; collision cylinder length=0.180 radius=0.025; visual cylinder length=0.180 radius=0.025
- added link arm_left_link_3, mass 0.120; collision cylinder length=0.180 radius=0.025; visual cylinder length=0.180 radius=0.025
- added link arm_left_link_4, mass 0.120; collision cylinder length=0.180 radius=0.025; visual cylinder length=0.180 radius=0.025
- added link arm_left_link_5, mass 0.120; collision cylinder length=0.180 radius=0.025; visual cylinder length=0.180 radius=0.025
- added link arm_left_link_6, mass 0.120; collision cylinder length=0.180 radius=0.025; visual cylinder length=0.180 radius=0.025
- added link arm_left_link_7, mass 0.120; collision cylinder length=0.180 radius=0.025; visual cylinder length=0.180 radius=0.025
- added link arm_right_link_1, mass 0.120; collision cylinder length=0.180 radius=0.025; visual cylinder length=0.180 radius=0.025
- added link arm_right_link_2, mass 0.120; collision cylinder length=0.180 radius=0.025; visual cylinder length=0.180 radius=0.025
- added link arm_right_link_3, mass 0.120; collision cylinder length=0.180 radius=0.025; visual cylinder length=0.180 radius=0.025
- added link arm_right_link_4, mass 0.120; collision cylinder length=0.180 radius=0.025; visual cylinder length=0.180 radius=0.025
- added link arm_right_link_5, mass 0.120; collision cylinder length=0.180 radius=0.025; visual cylinder length=0.180 radius=0.025
- added link arm_right_link_6, mass 0.120; collision cylinder length=0.180 radius=0.025; visual cylinder length=0.180 radius=0.025
- added link arm_right_link_7, mass 0.120; collision cylinder length=0.180 radius=0.025; visual cylinder length=0.180 radius=0.025
- added link neck_left_link_1, mass 0.080; collision cylinder length=0.080 radius=0.020; visual cylinder length=0.080 radius=0.020
- added link neck_left_link_2, mass 0.080; collision cylinder length=0.080 radius=0.020; visual cylinder length=0.080 radius=0.020
- added link neck_left_link_3, mass 0.080; collision cylinder length=0.080 radius=0.020; visual cylinder length=0.080 radius=0.020
- added link neck_left_link_4, mass 0.080; collision cylinder length=0.080 radius=0.020; visual cylinder length=0.080 radius=0.020
- added link neck_left_link_5, mass 0.080; collision cylinder length=0.080 radius=0.020; visual cylinder length=0.080 radius=0.020
- added link neck_left_link_6, mass 0.080; collision cylinder length=0.080 radius=0.020; visual cylinder length=0.080 radius=0.020
- added link neck_left_link_7, mass 0.080; collision cylinder length=0.080 radius=0.020; visual cylinder length=0.080 radius=0.020
- added link neck_mount_link, mass 0.200; collision sphere radius=0.050; visual sphere radius=0.050
- added link neck_right_link_1, mass 0.080; collision cylinder length=0.080 radius=0.020; visual cylinder length=0.080 radius=0.020
- added link neck_right_link_2, mass 0.080; collision cylinder length=0.080 radius=0.020; visual cylinder length=0.080 radius=0.020
- added link neck_right_link_3, mass 0.080; collision cylinder length=0.080 radius=0.020; visual cylinder length=0.080 radius=0.020
- added link neck_right_link_4, mass 0.080; collision cylinder length=0.080 radius=0.020; visual cylinder length=0.080 radius=0.020
- added link neck_right_link_5, mass 0.080; collision cylinder length=0.080 radius=0.020; visual cylinder length=0.080 radius=0.020
- added link neck_right_link_6, mass 0.080; collision cylinder length=0.080 radius=0.020; visual cylinder length=0.080 radius=0.020
- added link neck_right_link_7, mass 0.080; collision cylinder length=0.080 radius=0.020; visual cylinder length=0.080 radius=0.020
Joints:
- added joint arm_left_joint_1: type continuous, parent body, child arm_left_link_1, origin xyz=0.050 0.250 0.250 rpy=0 0 0, axis 0 0 1
- added joint arm_left_joint_2: type continuous, parent arm_left_link_1, child arm_left_link_2, origin xyz=0.000 0.000 0.180 rpy=0 0 0, axis 0 1 0
- added joint arm_left_joint_3: type continuous, parent arm_left_link_2, child arm_left_link_3, origin xyz=0.000 0.000 0.180 rpy=0 0 0, axis 0 1 0
- added joint arm_left_joint_4: type continuous, parent arm_left_link_3, child arm_left_link_4, origin xyz=0.000 0.000 0.180 rpy=0 0 0, axis 1 0 0
- added joint arm_left_joint_5: type continuous, parent arm_left_link_4, child arm_left_link_5, origin xyz=0.000 0.000 0.180 rpy=0 0 0, axis 0 1 0
- added joint arm_left_joint_6: type continuous, parent arm_left_link_5, child arm_left_link_6, origin xyz=0.000 0.000 0.180 rpy=0 0 0, axis 1 0 0
- added joint arm_left_joint_7: type continuous, parent arm_left_link_6, child arm_left_link_7, origin xyz=0.000 0.000 0.180 rpy=0 0 0, axis 0 1 0
- added joint arm_right_joint_1: type continuous, parent body, child arm_right_link_1, origin xyz=0.050 -0.250 0.250 rpy=0 0 0, axis 0 0 1
- added joint arm_right_joint_2: type continuous, parent arm_right_link_1, child arm_right_link_2, origin xyz=0.000 0.000 0.180 rpy=0 0 0, axis 0 1 0
- added joint arm_right_joint_3: type continuous, parent arm_right_link_2, child arm_right_link_3, origin xyz=0.000 0.000 0.180 rpy=0 0 0, axis 0 1 0
- added joint arm_right_joint_4: type continuous, parent arm_right_link_3, child arm_right_link_4, origin xyz=0.000 0.000 0.180 rpy=0 0 0, axis 1 0 0
- added joint arm_right_joint_5: type continuous, parent arm_right_link_4, child arm_right_link_5, origin xyz=0.000 0.000 0.180 rpy=0 0 0, axis 0 1 0
- added joint arm_right_joint_6: type continuous, parent arm_right_link_5, child arm_right_link_6, origin xyz=0.000 0.000 0.180 rpy=0 0 0, axis 1 0 0
- added joint arm_right_joint_7: type continuous, parent arm_right_link_6, child arm_right_link_7, origin xyz=0.000 0.000 0.180 rpy=0 0 0, axis 0 1 0
- added joint neck_left_joint_1: type continuous, parent neck_mount_link, child neck_left_link_1, origin xyz=0.000 0.060 0.000 rpy=0 0 0, axis 0 0 1
- added joint neck_left_joint_2: type continuous, parent neck_left_link_1, child neck_left_link_2, origin xyz=0.000 0.000 0.080 rpy=0 0 0, axis 0 1 0
- added joint neck_left_joint_3: type continuous, parent neck_left_link_2, child neck_left_link_3, origin xyz=0.000 0.000 0.080 rpy=0 0 0, axis 1 0 0
- added joint neck_left_joint_4: type continuous, parent neck_left_link_3, child neck_left_link_4, origin xyz=0.000 0.000 0.080 rpy=0 0 0, axis 0 1 0
- added joint neck_left_joint_5: type continuous, parent neck_left_link_4, child neck_left_link_5, origin xyz=0.000 0.000 0.080 rpy=0 0 0, axis 1 0 0
- added joint neck_left_joint_6: type continuous, parent neck_left_link_5, child neck_left_link_6, origin xyz=0.000 0.000 0.080 rpy=0 0 0, axis 0 1 0
- added joint neck_left_joint_7: type continuous, parent neck_left_link_6, child neck_left_link_7, origin xyz=0.000 0.000 0.080 rpy=0 0 0, axis 1 0 0
- added joint neck_mount_fixed: type fixed, parent body, child neck_mount_link, origin xyz=0 0 0.45 rpy=0 0 0
- added joint neck_right_joint_1: type continuous, parent neck_mount_link, child neck_right_link_1, origin xyz=0.000 -0.060 0.000 rpy=0 0 0, axis 0 0 1
- added joint neck_right_joint_2: type continuous, parent neck_right_link_1, child neck_right_link_2, origin xyz=0.000 0.000 0.080 rpy=0 0 0, axis 0 1 0
- added joint neck_right_joint_3: type continuous, parent neck_right_link_2, child neck_right_link_3, origin xyz=0.000 0.000 0.080 rpy=0 0 0, axis 1 0 0
- added joint neck_right_joint_4: type continuous, parent neck_right_link_3, child neck_right_link_4, origin xyz=0.000 0.000 0.080 rpy=0 0 0, axis 0 1 0
- added joint neck_right_joint_5: type continuous, parent neck_right_link_4, child neck_right_link_5, origin xyz=0.000 0.000 0.080 rpy=0 0 0, axis 1 0 0
- added joint neck_right_joint_6: type continuous, parent neck_right_link_5, child neck_right_link_6, origin xyz=0.000 0.000 0.080 rpy=0 0 0, axis 0 1 0
- added joint neck_right_joint_7: type continuous, parent neck_right_link_6, child neck_right_link_7, origin xyz=0.000 0.000 0.080 rpy=0 0 0, axis 1 0 0
