Commit message: Fix hardware launch parameter loading and document modular toggles

File: src/legged_examples/legged_dm_description/urdf/dm.urdf (robot description, URDF)
Before this commit: robot legged_dm_description_no_arm, 21 links, 20 joints
Links:
- removed link leg_l1_link
- removed link leg_l2_link
- removed link leg_l3_link
- removed link leg_l4_link
- removed link leg_l5_link
- removed link leg_l6_link
- removed link leg_l7_link
- removed link leg_l_f1_link
- removed link leg_l_f2_link
- removed link leg_r1_link
- removed link leg_r2_link
- removed link leg_r3_link
- removed link leg_r4_link
- removed link leg_r5_link
- removed link leg_r6_link
- removed link leg_r7_link
- removed link leg_r_f1_link
- removed link leg_r_f2_link
- added link leg_left_f1_link, mass 0.01; collision sphere radius=0.001; visual sphere radius=0.001
- added link leg_left_f2_link, mass 0.01; collision sphere radius=0.001; visual sphere radius=0.001
- added link leg_left_link_1, mass 0.492347; collision box size=0.0001 0.0001 0.0001; visual mesh filename=package://legged_dm_description/meshes/leg_left_link_1.STL
- added link leg_left_link_2, mass 0.11551; collision box size=0.0001 0.0001 0.0001; visual mesh filename=package://legged_dm_description/meshes/leg_left_link_2.STL
- added link leg_left_link_3, mass 0.921105; collision box size=0.0001 0.0001 0.0001; visual mesh filename=package://legged_dm_description/meshes/leg_left_link_3.STL
- added link leg_left_link_4, mass 0.519684; collision box size=0.041 0.07 0.15; visual mesh filename=package://legged_dm_description/meshes/leg_left_link_4.STL
- added link leg_left_link_5, mass 0.172725; collision box size=0.175 0.06 0.02; visual mesh filename=package://legged_dm_description/meshes/leg_left_link_5.STL
- added link leg_left_link_6, mass 0.01; collision sphere radius=0.001; visual sphere radius=0.001
- added link leg_left_link_7, mass 0.01; collision sphere radius=0.001; visual sphere radius=0.001
- added link leg_right_f1_link, mass 0.01; collision sphere radius=0.001; visual sphere radius=0.001
- added link leg_right_f2_link, mass 0.01; collision sphere radius=0.001; visual sphere radius=0.001
- added link leg_right_link_1, mass 0.4921; collision box size=0.0001 0.0001 0.0001; visual mesh filename=package://legged_dm_description/meshes/leg_right_link_1.STL
- added link leg_right_link_2, mass 0.115510; collision box size=0.0001 0.0001 0.0001; visual mesh filename=package://legged_dm_description/meshes/leg_right_link_2.STL
- added link leg_right_link_3, mass 0.921105; collision box size=0.0001 0.0001 0.0001; visual mesh filename=package://legged_dm_description/meshes/leg_right_link_3.STL
- added link leg_right_link_4, mass 0.519684; collision box size=0.041 0.07 0.15; visual mesh filename=package://legged_dm_description/meshes/leg_right_link_4.STL
- added link leg_right_link_5, mass 0.172725; collision box size=0.175 0.06 0.02; visual mesh filename=package://legged_dm_description/meshes/leg_right_link_5.STL
- added link leg_right_link_6, mass 0.01; collision sphere radius=0.001; visual sphere radius=0.001
- added link leg_right_link_7, mass 0.01; collision sphere radius=0.001; visual sphere radius=0.001
Joints:
- removed joint leg_l1_joint
- removed joint leg_l2_joint
- removed joint leg_l3_joint
- removed joint leg_l4_joint
- removed joint leg_l5_fixed_1
- removed joint leg_l5_fixed_2
- removed joint leg_l5_joint
- removed joint leg_l6_joint
- removed joint leg_l7_joint
- removed joint leg_r1_joint
- removed joint leg_r2_joint
- removed joint leg_r3_joint
- removed joint leg_r4_joint
- removed joint leg_r5_fixed_1
- removed joint leg_r5_fixed_2
- removed joint leg_r5_joint
- removed joint leg_r6_joint
- removed joint leg_r7_joint
- added joint leg_left_fixed_1: type fixed, parent leg_left_link_5, child leg_left_f1_link, origin xyz=0.113 -0.008 -0.006 rpy=0 0 0
- added joint leg_left_fixed_2: type fixed, parent leg_left_link_5, child leg_left_f2_link, origin xyz=-0.061 -0.008 -0.006 rpy=0 0 0
- added joint leg_left_joint_1: type revolute, parent loin_yaw_Link, child leg_left_link_1, origin xyz=3.7385E-05 0.05355 -0.062 rpy=0 0 0, axis 0 1 0, limit lower=-1.05 upper=1.05 effort=26 velocity=10
- added joint leg_left_joint_2: type revolute, parent leg_left_link_1, child leg_left_link_2, origin xyz=0.031079 0.041978 0 rpy=0 0 0, axis 1 0 0, limit lower=-0.52 upper=0.785 effort=26 velocity=10
- added joint leg_left_joint_3: type revolute, parent leg_left_link_2, child leg_left_link_3, origin xyz=-0.03105 2.1677E-05 -0.07405 rpy=0 0 0, axis 0 0 1, limit lower=-0.52 upper=0.785 effort=26 velocity=10
- added joint leg_left_joint_4: type revolute, parent leg_left_link_3, child leg_left_link_4, origin xyz=2.1677E-05 0.03105 -0.11705 rpy=0 0 0, axis 0 1 0, limit lower=-0.3 upper=2.3562 effort=26 velocity=10
- added joint leg_left_joint_5: type revolute, parent leg_left_link_4, child leg_left_link_5, origin xyz=-3.1151E-05 -0.02305 -0.2 rpy=0 0 0, axis 0 1 0, limit lower=-1.047 upper=0.3 effort=26 velocity=10
- added joint leg_left_joint_6: type revolute, parent leg_left_link_5, child leg_left_link_6, origin xyz=0 0 0 rpy=0 0 0, axis 0 1 0, limit lower=-1.57 upper=1.57 effort=26 velocity=10
- added joint leg_left_joint_7: type revolute, parent leg_left_link_6, child leg_left_link_7, origin xyz=0 0 0 rpy=0 0 0, axis 0 1 0, limit lower=-1.57 upper=1.57 effort=26 velocity=10
- added joint leg_right_fixed_1: type fixed, parent leg_right_link_5, child leg_right_f1_link, origin xyz=0.113 0.008 -0.006 rpy=0 0 0
- added joint leg_right_fixed_2: type fixed, parent leg_right_link_5, child leg_right_f2_link, origin xyz=-0.061 0.008 -0.006 rpy=0 0 0
- added joint leg_right_joint_1: type revolute, parent loin_yaw_Link, child leg_right_link_1, origin xyz=-3.7385E-05 -0.05355 -0.062 rpy=0 0 0, axis 0 1 0, limit lower=-1.05 upper=1.05 effort=26 velocity=10
- added joint leg_right_joint_2: type revolute, parent leg_right_link_1, child leg_right_link_2, origin xyz=0.031021 -0.042022 0 rpy=0 0 0, axis 1 0 0, limit lower=-0.785 upper=0.52 effort=26 velocity=10
- added joint leg_right_joint_3: type revolute, parent leg_right_link_2, child leg_right_link_3, origin xyz=-0.03105 2.1677E-05 -0.07405 rpy=0 0 0, axis 0 0 1, limit lower=-0.785 upper=0.52 effort=26 velocity=10
- added joint leg_right_joint_4: type revolute, parent leg_right_link_3, child leg_right_link_4, origin xyz=-2.1677E-05 -0.03105 -0.11705 rpy=0 0 0, axis 0 1 0, limit lower=-0.3 upper=2.3562 effort=26 velocity=10
- added joint leg_right_joint_5: type revolute, parent leg_right_link_4, child leg_right_link_5, origin xyz=1.6127E-05 0.0231 -0.2 rpy=0 0 0, axis 0 1 0, limit lower=-1.047 upper=0.3 effort=26 velocity=10
- added joint leg_right_joint_6: type revolute, parent leg_right_link_5, child leg_right_link_6, origin xyz=0 0 0 rpy=0 0 0, axis 0 1 0, limit lower=-1.57 upper=1.57 effort=26 velocity=10
- added joint leg_right_joint_7: type revolute, parent leg_right_link_6, child leg_right_link_7, origin xyz=0 0 0 rpy=0 0 0, axis 0 1 0, limit lower=-1.57 upper=1.57 effort=26 velocity=10

File: src/right_arm_moveit_config/config/gazebo_wanren_arm.urdf (robot description, URDF)
Before this commit: robot wanren_arm, 8 links, 7 joints
Links:
- removed link body
- removed link leg_r1_link
- removed link leg_r2_link
- removed link leg_r3_link
- removed link leg_r4_link
- removed link leg_r5_link
- removed link leg_r6_link
- removed link leg_r7_link
- added link leg_right_link_1, mass 0.292899916417866; collision mesh filename=package://wanren_arm/meshes/leg_r1.STL; visual mesh filename=package://wanren_arm/meshes/leg_r1.STL
- added link leg_right_link_2, mass 0.118782011304387; collision mesh filename=package://wanren_arm/meshes/leg_r2.STL; visual mesh filename=package://wanren_arm/meshes/leg_r2.STL
- added link leg_right_link_3, mass 0.395227613542105; collision mesh filename=package://wanren_arm/meshes/leg_r3.STL; visual mesh filename=package://wanren_arm/meshes/leg_r3.STL
- added link leg_right_link_4, mass 0.0222841339329651; collision mesh filename=package://wanren_arm/meshes/leg_r4.STL; visual mesh filename=package://wanren_arm/meshes/leg_r4.STL
- added link leg_right_link_5, mass 0.38824624930896; collision mesh filename=package://wanren_arm/meshes/leg_r5.STL; visual mesh filename=package://wanren_arm/meshes/leg_r5.STL
- added link leg_right_link_6, mass 0.174871084341935; collision mesh filename=package://wanren_arm/meshes/leg_r6.STL; visual mesh filename=package://wanren_arm/meshes/leg_r6.STL
- added link leg_right_link_7, mass 0.784412251530751; collision box size=0.1 0.05 0.04; visual mesh filename=package://wanren_arm/meshes/leg_r7.STL
- added link torso_link, mass 0.60016209200883; collision mesh filename=package://wanren_arm/meshes/body.STL; visual mesh filename=package://wanren_arm/meshes/body.STL
Joints:
- removed joint leg_r1_joint
- removed joint leg_r2_joint
- removed joint leg_r3_joint
- removed joint leg_r4_joint
- removed joint leg_r5_joint
- removed joint leg_r6_joint
- removed joint leg_r7_joint
- added joint leg_right_joint_1: type continuous, parent torso_link, child leg_right_link_1, origin xyz=0 0 0.011999999999999 rpy=0 0 0, axis 0 0 -1
- added joint leg_right_joint_2: type continuous, parent leg_right_link_1, child leg_right_link_2, origin xyz=-0.0136812977041495 -0.0436944371355362 0.0808116620061236 rpy=0 0 0, axis 0.29752487908452 0.954714065218347 0
- added joint leg_right_joint_3: type continuous, parent leg_right_link_2, child leg_right_link_3, origin xyz=0.0412068272569313 0.104588881771451 0.106228185949221 rpy=0 0 0, axis -0.0722349306802614 0.022511126419206 -0.997133573788866
- added joint leg_right_joint_4: type continuous, parent leg_right_link_3, child leg_right_link_4, origin xyz=-0.00228042956033238 -0.0297792321778995 0.0833604475054363 rpy=0 0 0, axis 0.282983296167026 0.959124144572578 0.0011529910516605
- added joint leg_right_joint_5: type continuous, parent leg_right_link_4, child leg_right_link_5, origin xyz=0.0181511434262854 0.025007599076044 0.111134888878763 rpy=0 1.26722046551249 0, axis 0.923719785557326 0.0273056458564005 -0.382094437900229
- added joint leg_right_joint_6: type continuous, parent leg_right_link_5, child leg_right_link_6, origin xyz=-0.0550712045826083 -0.0332459772838745 -0.000878918231283499 rpy=1.5372364468678 -1.26722046551249 0, axis 0.565655964466871 0 -0.824641334073823
- added joint leg_right_joint_7: type continuous, parent leg_right_link_6, child leg_right_link_7, origin xyz=0.0506954674848457 0.0975609362242854 -0.0679978120533321 rpy=-1.5372364468678 0 0, axis 0.804819794366103 -0.559061164385712 -0.199288015375224

File: src/wanren_arm/urdf/wanren_arm.urdf (robot description, URDF)
Before this commit: robot wanren_arm, 44 links, 43 joints
Links:
- removed link arm_left_link_1
- removed link arm_left_link_2
- removed link arm_left_link_3
- removed link arm_left_link_4
- removed link arm_left_link_5
- removed link arm_left_link_6
- removed link arm_left_link_7
- removed link arm_right_link_1
- removed link arm_right_link_2
- removed link arm_right_link_3
- removed link arm_right_link_4
- removed link arm_right_link_5
- removed link arm_right_link_6
- removed link arm_right_link_7
- removed link body
- removed link leg_l1_link
- removed link leg_l2_link
- removed link leg_l3_link
- removed link leg_l4_link
- removed link leg_l5_link
- removed link leg_l6_link
- removed link leg_l7_link
- removed link leg_r1_link
- removed link leg_r2_link
- removed link leg_r3_link
- removed link leg_r4_link
- removed link leg_r5_link
- removed link leg_r6_link
- removed link leg_r7_link
- removed link neck_left_link_1
- removed link neck_left_link_2
- removed link neck_left_link_3
- removed link neck_left_link_4
- removed link neck_left_link_5
- removed link neck_left_link_6
- removed link neck_left_link_7
- removed link neck_mount_link
- removed link neck_right_link_1
- removed link neck_right_link_2
- removed link neck_right_link_3
- removed link neck_right_link_4
- removed link neck_right_link_5
- removed link neck_right_link_6
- removed link neck_right_link_7
- added link base_link, mass 0.001
- added link torso_link, mass 0.60016209200883; collision mesh filename=package://wanren_arm/meshes/body.STL; visual mesh filename=package://wanren_arm/meshes/body.STL
Joints:
- removed joint arm_left_joint_1
- removed joint arm_left_joint_2
- removed joint arm_left_joint_3
- removed joint arm_left_joint_4
- removed joint arm_left_joint_5
- removed joint arm_left_joint_6
- removed joint arm_left_joint_7
- removed joint arm_right_joint_1
- removed joint arm_right_joint_2
- removed joint arm_right_joint_3
- removed joint arm_right_joint_4
- removed joint arm_right_joint_5
- removed joint arm_right_joint_6
- removed joint arm_right_joint_7
- removed joint leg_l1_joint
- removed joint leg_l2_joint
- removed joint leg_l3_joint
- removed joint leg_l4_joint
- removed joint leg_l5_joint
- removed joint leg_l6_joint
- removed joint leg_l7_joint
- removed joint leg_r1_joint
- removed joint leg_r2_joint
- removed joint leg_r3_joint
- removed joint leg_r4_joint
- removed joint leg_r5_joint
- removed joint leg_r6_joint
- removed joint leg_r7_joint
- removed joint neck_left_joint_1
- removed joint neck_left_joint_2
- removed joint neck_left_joint_3
- removed joint neck_left_joint_4
- removed joint neck_left_joint_5
- removed joint neck_left_joint_6
- removed joint neck_left_joint_7
- removed joint neck_mount_fixed
- removed joint neck_right_joint_1
- removed joint neck_right_joint_2
- removed joint neck_right_joint_3
- removed joint neck_right_joint_4
- removed joint neck_right_joint_5
- removed joint neck_right_joint_6
- removed joint neck_right_joint_7
